Commit message: Feat: add pkg:realsense_ros_gazebo and modify omni.gazebo.xacro. now the robot can publish depth topic

File: OpenBase/ROS/open_base/xacro/omni.gazebo.xacro (robot description, xacro)
@@ -63,3 +63,7 @@
     </sensor>
   </gazebo>
+  <xacro:include filename="$(find realsense_ros_gazebo)/xacro/depthcam.xacro"/>
+  <xacro:realsense_d435 sensor_name="d435" parent_link="base_link" rate="10">
+    <origin rpy="0 0 0 " xyz="0 0 0.4"/>
+  </xacro:realsense_d435>
 </robot>
